File: schematics/mainboard/mainboard.sch (EAGLE design)
At the start: 67 parts, among them IC1 OPA2344P, IC2 74AHC00D, IC3 LM2576-5.0, IC4 LM2576-3.3, Q1 BD140, Q2 BD140, Q3 IRF540, U1 STM32F777VIT

Commit message: Add files via upload
Parts:
- added C22, C23: 2u2, rcl:C-EUC0805
- added C24, C25: 100n, rcl:C-EUC0805
- added JP3: SWD, pinhead:PINHD-1X5/90
- added L10, L9: (no value), inductor-neosid:SM-B5
- added OS1: ECS-3225MV-160-CN-TR, IQD-Frequency-Products:OSC-OE-CFPS-39
Connections:
- new net DAC_OUT: U1.P$28
- new net N$24: C22.1, U1.P$48
- new net N$25: C23.1, U1.P$73
- new net NRST: JP3.2, U1.P$14
- new net OSC_IN: OS1.OUT, U1.P$12
- new net SWCLK: JP3.3, U1.P$76
- new net SWDIO: JP3.4, U1.P$72
- new net VDDA: C24.1, L10.2, U1.P$21
- new net VREF: C25.1, L9.2, U1.P$20
- net +3V3: now also JP3.5, L10.1, L9.1, OS1.VDD, U1.P$100, U1.P$11, U1.P$27, U1.P$50, U1.P$6, U1.P$75
- net GND: now also C22.2, C23.2, C24.2, C25.2, JP3.1, OS1.VSS, U1.P$10, U1.P$19, U1.P$26, U1.P$49, U1.P$74, U1.P$94, U1.P$99
- net LCD_PWM: now also U1.P$59

Commit message: Add files via upload
Parts:
- added JP1, JP2: (no value), pinhead:PINHD-1X3
Connections:
- net GND: now also JP1.3, JP2.3
- net N$15: now also JP1.1
- net N$19: now also JP2.1
- net TACHO_FAN_L: now also JP2.2
- net TACHO_FAN_R: now also JP1.2
Other:
- moved on the sheet: C10, C3, C4, C9, IC1A, IC1B, Q1, Q2, R1, R10, R11, R12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

Commit message: Add files via upload
Parts:
- added C26, C27: 22u/25, rcl:CPOL-EUE2-5
- added C28, C29: 100n, rcl:C-EUC0805
- added C30: 4.7u, rcl:C-EUC0805
- added IC5: LM339N, linear:LM339N
- added R20, R21, R25: 4k7, resistor:R-EU_R0805
- added R22: 2k7, resistor:R-EU_R0805
- added R23, R24: (no value), rcl:R-TRIMM3296W
- R17: value 4k7 -> 2k7
Connections:
- new net L_FAN_OK: IC5A.OUT, IC5B.OUT, R20.2
- new net N$26: C26.+, IC5C.+IN, IC5D.+IN, R16.1, R17.2
- new net N$27: C27.+, IC5A.-IN, IC5B.+IN, R21.1, R22.2
- new net R_FAN_OK: IC5C.OUT, IC5D.OUT, R25.2
- new net V_DN: C29.1, IC5B.-IN, IC5D.-IN, R23.S
- new net V_UP: C28.1, IC5A.+IN, IC5C.-IN, R24.S
- net +3V3: now also C30.1, IC5P.V+, R20.1, R22.1, R23.E, R24.E, R25.1; no longer R16.1
- net GND: now also C26.-, C27.-, C28.2, C29.2, C30.2, IC5P.GND, R23.A, R24.A
- net TACHO_FAN_L: now also R21.2; no longer R16.2
- net TACHO_FAN_R: now also R16.2; no longer R17.2
Other:
- moved on the sheet: R16, R17

Commit message: Add files via upload
Parts:
- added C31: 4.7u, rcl:C-EUC0805
- C10, C9: value 1u -> 100n
- C11, C12: value 100n -> 1u
- C17, C18: value 100u/35V -> 100n; device rcl:CPOL-EUE3.5-8 -> rcl:C-EUC0805
- C19: value 1000u/10V -> 100n; device rcl:CPOL-EUE3.5-8 -> rcl:C-EUC0805
- C20: value 1000u/10V -> 10n; device rcl:CPOL-EUE3.5-8 -> rcl:C-EUC0805
- C22, C23: value 2u2 -> 100n
- C24, C25: value 100n -> 100u/35V; device rcl:C-EUC0805 -> rcl:CPOL-EUE3.5-8
- C26, C27: value 22u/25 -> 1000u/10V; device rcl:CPOL-EUE2-5 -> rcl:CPOL-EUE3.5-8
- C28, C29: value 100n -> 2u2
- C30: value 4.7u -> 100n
- C5, C6: value 100n -> 22u/25; device rcl:C-EUC0805 -> rcl:CPOL-EUE2-5
- IC2: value 74AHC00D -> LM339N; device 74xx-eu:7400D -> linear:LM339N
- IC3: value LM2576-5.0 -> 74AHC00D; device v-reg-3:LM2576S -> 74xx-eu:7400D
- IC5: value LM339N -> LM2576-5.0; device linear:LM339N -> v-reg-3:LM2576S
- L10, L9: value (none) -> 100u/5A; device inductor-neosid:SM-B5 -> rcl:L-EUTJ5-U2
- L7, L8: value 100u/5A -> (none); device rcl:L-EUTJ5-U2 -> inductor-neosid:SM-B5
- R10, R11, R15: value 10k -> 4k7
- R12, R13: value 4k7 -> 10k
- R14: value 100R -> 4k7
- R16: value 4k7 -> 2k7
- R18: value 22k -> 100R
- R19: value 22k -> 10k
- R20, R21: value 4k7 -> 22k
- R22: value 2k7 -> 4k7
- R23: value (none) -> 4k7; device rcl:R-TRIMM3296W -> resistor:R-EU_R0805
- R25: value 4k7 -> (none); device resistor:R-EU_R0805 -> rcl:R-TRIMM3296W
- renumbered IC4 to IC6
Connections:
- net +12V: now also C24.+, C25.+, IC5.VIN, R12.2, R13.2; no longer C17.+, C18.+, IC3.VIN, R10.2, R11.2
- net +3V3: now also C13.1, C20.1, C26.+, C31.1, C8.1, IC2P.V+, IC3A.I0, IC3B.I1, IC3P.VCC, L7.1, L8.1, L9.2, R16.1, R23.1, R25.E; no longer C11.1, C16.1, C19.+, C6.1, IC2A.I0, IC2C.I0, IC2P.VCC, IC5P.V+, L10.1, L7.2, L9.1, R20.1, R23.E, R25.1
- net +5V: now also C10.2, C17.2, C27.+, IC5.FB, L10.2; no longer C13.2, C20.+, C8.2, IC3.FB, L8.2
- net 32M_REF_IN_RX: now also IC3B.O; no longer IC2C.O
- net 32M_REF_IN_TX: now also IC3A.O; no longer IC2A.O
- net 32M_REF_OUT: now also IC3A.I1, IC3B.I0; no longer IC2A.I1, IC2C.I1
- net GND: now also C10.1, C13.2, C14.2, C15.2, C17.1, C18.1, C19.1, C20.2, C24.-, C25.-, C31.2, C5.-, C6.-, C8.2, C9.1, IC3C.I0, IC3C.I1, IC3D.I0, IC3D.I1, IC3P.GND, IC5.GND, IC5.OFF, R19.2, R25.A; no longer C10.2, C13.1, C14.1, C15.1, C17.-, C18.-, C19.-, C20.-, C24.2, C25.2, C5.1, C6.2, C8.1, C9.2, IC2B.I0, IC2B.I1, IC2D.I0, IC2D.I1, IC3.GND, IC3.OFF, IC5P.GND, R15.2, R23.A
- net LCD_PWM: now also R18.2; no longer R14.2
- net L_FAN_OK: now also IC2A.OUT, IC2B.OUT, R22.2; no longer IC5A.OUT, IC5B.OUT, R20.2
- net N$1: now also IC5.OUT, L10.1; no longer IC3.OUT, L8.1
- net N$11: now also C12.1, R21.2; no longer C10.1, R19.2
- net N$12: now also R12.1; no longer R10.1
- net N$13: now also C9.2; no longer C7.2
- net N$17: now also R13.1; no longer R11.1
- net N$18: now also R14.1; no longer R12.1
- net N$2: now also R18.1, R19.1; no longer R14.1, R15.1
- net N$21: now also R14.2; no longer R12.2
- net N$22: now also R15.1; no longer R13.1
- net N$23: now also R15.2; no longer R13.2
- net N$24: now also C28.1; no longer C22.1
- net N$25: now also C29.1; no longer C23.1
- net N$26: now also C6.+, IC2C.+IN, IC2D.+IN, R11.1; no longer C26.+, IC5C.+IN, IC5D.+IN, R16.1
- net N$27: now also C5.+, IC2A.-IN, IC2B.+IN, R10.1, R16.2; no longer C27.+, IC5A.-IN, IC5B.+IN, R21.1, R22.2
- net N$3: now also L9.1; no longer L7.1
- net N$4: now also C14.1; no longer C12.1
- net N$5: now also C18.2; no longer C14.2
- net N$6: now also C19.2; no longer C15.2
- net N$8: now also C7.2; no longer C5.2
- net N$9: now also C11.1, R20.2; no longer C9.1, R18.2
- net PWM_FAN_L: now also R20.1; no longer R18.1
- net PWM_FAN_R: now also R21.1; no longer R19.1
- net R_FAN_OK: now also IC2C.OUT, IC2D.OUT, R23.2; no longer IC5C.OUT, IC5D.OUT, R25.2
- net TACHO_FAN_L: now also R10.2; no longer R21.2
- net TACHO_FAN_R: now also R11.2; no longer R16.2
- net VDDA: now also C22.1, L8.2; no longer C24.1, L10.2
- net VREF: now also C23.1, L7.2; no longer C25.1, L9.2
- net V_DN: now also C16.1, IC2B.-IN, IC2D.-IN, R25.S; no longer C29.1, IC5B.-IN, IC5D.-IN, R23.S
- net V_UP: now also C15.1, IC2A.+IN, IC2C.-IN; no longer C28.1, IC5A.+IN, IC5C.-IN
Other:
- moved on the sheet: C10, C11, C12, C13, C14, C15, C16, C21, C22, C23, C26, C27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

Commit message: Add files via upload
Parts:
- added D3: 1N4148, diode:1N4148DO35-7
- added R27: (no value), pot:TRIM_EU-CA6V
Connections:
- new net ANALOG_IN_0: U1.P$22
- new net ANALOG_IN_1: U1.P$23
- new net ANALOG_IN_2: U1.P$24
- new net ANALOG_IN_3: U1.P$25
- new net LED_0: U1.P$77
- new net LED_1: U1.P$78
- new net LED_2: U1.P$79
- new net LED_3: U1.P$80
- new net LED_4: U1.P$81
- new net LED_5: U1.P$82
- new net PTT: U1.P$97
- new net USART1_RX: U1.P$69
- new net USART1_TX: U1.P$68
- net +5V: now also R27.E
- net GND: now also R27.A
- net LCD_A: now also D3.C
- net LCD_CONTR: now also R27.S
- net LCD_DB0: now also U1.P$38
- net LCD_DB1: now also U1.P$39
- net LCD_DB2: now also U1.P$40
- net LCD_DB3: now also U1.P$41
- net LCD_DB4: now also U1.P$42
- net LCD_DB5: now also U1.P$43
- net LCD_DB6: now also U1.P$44
- net LCD_DB7: now also U1.P$45
- net LCD_E: now also U1.P$37
- net LCD_K: now also D3.A
- net LCD_RES: now also U1.P$46
- net LCD_RS: now also U1.P$35
- net LCD_RW: now also U1.P$36
- net RX_CS: now also U1.P$32
- net RX_MISO: now also U1.P$30
- net RX_MOSI: now also U1.P$31
- net RX_NIRQ: now also U1.P$33
- net RX_SCK: now also U1.P$29
- net RX_SDN: now also U1.P$34
- net TX_CS: now also U1.P$55
- net TX_MISO: now also U1.P$53
- net TX_MOSI: now also U1.P$54
- net TX_NIRQ: now also U1.P$56
- net TX_SCK: now also U1.P$52
- net TX_SDN: now also U1.P$51

Commit message: Add files via upload
Parts:
- added C32: 22u/25, rcl:CPOL-EUE2-5
- added JP4: LEDS, pinhead:PINHD-2X6
- added JP5: KBD, pinhead:PINHD-1X5
- added JP6: TAMPER, pinhead:PINHD-1X2
- added R26, R28, R29, R30, R31, R32, R39, R40, R41, R42, R43: 4k7, resistor:R-EU_R0805
- added R33, R34, R35, R36, R37, R38: 820R, resistor:R-EU_R0805
- added T3, T4, T5, T6, T7, T8: BC847, transistor:BC847
- JP3: device pinhead:PINHD-1X5/90 -> pinhead:PINHD-1X5
Connections:
- new net BTN_0: JP5.1, R39.2, U1.P$83
- new net BTN_1: JP5.2, R40.2, U1.P$84
- new net BTN_2: JP5.3, R41.2, U1.P$85
- new net BTN_3: JP5.4, R42.2, U1.P$88
- new net ENC_A: U1.P$91
- new net ENC_B: U1.P$90
- new net ENC_BTN: U1.P$98
- new net N$28: R26.2, T3.B
- new net N$29: R33.1, T3.C
- new net N$30: JP4.1, R33.2
- new net N$31: JP4.3, R34.2
- new net N$32: R28.2, T4.B
- new net N$33: R34.1, T4.C
- new net N$34: JP4.5, R35.2
- new net N$35: R29.2, T5.B
- new net N$36: R35.1, T5.C
- new net N$37: JP4.7, R36.2
- new net N$38: R30.2, T6.B
- new net N$39: R36.1, T6.C
- new net N$40: JP4.9, R37.2
- new net N$41: R31.2, T7.B
- new net N$42: R37.1, T7.C
- new net N$43: JP4.11, R38.2
- new net N$44: R32.2, T8.B
- new net N$46: R38.1, T8.C
- new net TAMPER: JP6.1, R43.2, U1.P$5
- net +12V: now also C32.+
- net +3V3: now also R39.1, R40.1, R41.1, R42.1, R43.1
- net +5V: now also JP4.10, JP4.12, JP4.2, JP4.4, JP4.6, JP4.8
- net GND: now also C32.-, JP5.5, JP6.2, T3.E, T4.E, T5.E, T6.E, T7.E, T8.E
- net LED_0: now also R26.1
- net LED_1: now also R28.1
- net LED_2: now also R29.1
- net LED_3: now also R30.1
- net LED_4: now also R31.1
- net LED_5: now also R32.1

Commit message: Add files via upload
Parts:
- added C33, C34: 10u/TA, resistor:C-EUC1206
Connections:
- net +3V3: now also C33.1, C34.1
- net GND: now also C33.2, C34.2
Other:
- moved on the sheet: C28, C29, U1

Commit message: Add files via upload
Connections:
- net 32M_REF_IN_RX: now also SV2.7; no longer SV2.2
- net 32M_REF_IN_TX: now also SV5.7; no longer SV5.2
- net GND: now also SV2.2, SV5.2; no longer SV2.1, SV5.1
- net RX_CS: now also SV2.5; no longer SV2.7
- net RX_MISO: now also SV2.3; no longer SV2.8
- net RX_NIRQ: now also SV2.1; no longer SV2.5
- net RX_SDN: now also SV2.8; no longer SV2.3
- net TX_CS: now also SV5.5; no longer SV5.7
- net TX_MISO: now also SV5.3; no longer SV5.8
- net TX_NIRQ: now also SV5.1; no longer SV5.5
- net TX_SDN: now also SV5.8; no longer SV5.3
