File: schematics/mainboard/mainboard.sch (EAGLE design)
At the start: 121 parts, among them IC1 OPA2344P, IC2 LM339N, IC3 74AHC00D, IC5 LM2576-5.0, IC6 LM2576-3.3, Q1 BD140, Q2 BD140, Q3 IRF540, T3 BC847, T4 BC847, T5 BC847, T6 BC847, T7 BC847, T8 BC847, U1 STM32F777VIT

Commit message: Add files via upload
Parts:
- removed IC6: LM2576-3.3, v-reg-3:LM2576S
- added C35: 100n, rcl:C-EUC0805
- added IC4: LM2576-5.0, v-reg-3:LM2576S
- C26, C27: value 1000u/10V -> 10u/TA; device rcl:CPOL-EUE3.5-8 -> resistor:C-EUC1206
- C28, C29: value 2u2 -> 1000u/10V; device rcl:C-EUC0805 -> rcl:CPOL-EUE3.5-8
- C30: value 100n -> 2u2
- C31: value 4.7u -> 100n
- C32: value 22u/25 -> 2u2; device rcl:CPOL-EUE2-5 -> rcl:C-EUC0805
- C33: value 10u/TA -> 4.7u; device resistor:C-EUC1206 -> rcl:C-EUC0805
- C34: value 10u/TA -> 22u/25; device resistor:C-EUC1206 -> rcl:CPOL-EUE2-5
- D1: value 1N5822 -> 1N4148; device diode:1N5819-T -> diode:1N4148DO35-7
- D3: value 1N4148 -> 1N5822; device diode:1N4148DO35-7 -> diode:1N5819-T
- IC1: value OPA2344P -> LM358N; device linear:OPA2344P -> linear:LM358N
- IC5: value LM2576-5.0 -> LM2576-3.3
- JP3: value SWD -> LEDS; device pinhead:PINHD-1X5 -> pinhead:PINHD-2X6
- JP4: value LEDS -> SWD; device pinhead:PINHD-2X6 -> pinhead:PINHD-1X5
- R1: value 10k -> (none); device resistor:R-EU_R0805 -> pot:TRIM_EU-CA6V
- R10: value 4k7 -> 470R
- R12: value 10k -> 4k7
- R14: value 4k7 -> 10k
- R16: value 2k7 -> 4k7
- R18: value 100R -> 2k7
- R19: value 10k -> 100R
- R2, R4: value 1k -> 10k
- R20: value 22k -> 10k
- R22: value 4k7 -> 22k
- R24: value (none) -> 4k7; device rcl:R-TRIMM3296W -> resistor:R-EU_R0805
- R26: value 4k7 -> (none); device resistor:R-EU_R0805 -> rcl:R-TRIMM3296W
- R27: value (none) -> 4k7; device pot:TRIM_EU-CA6V -> resistor:R-EU_R0805
- R28, R30, R32: value 4k7 -> 820R
- R3: value 10k -> 1k
- R33, R35, R37: value 820R -> 4k7
- R5: value 2k7 -> 1k
- R7: value 0R -> 2k7
- R8: value 470R -> 0R
- T1, T2: value (none) -> 2N3904
Connections:
- net +12V: now also C34.+, IC1P.V+, IC4.VIN, R14.2; no longer C32.+, IC1A.V+, IC6.VIN, R12.2
- net +3V3: now also C26.1, C27.1, C28.+, IC5.FB, JP4.5, R18.1, R24.1, R26.E; no longer C26.+, C30.1, C34.1, IC6.FB, JP3.5, R16.1, R22.1, R24.E
- net +5V: now also C29.+, IC4.FB, JP3.10, JP3.12, JP3.2, JP3.4, JP3.6, JP3.8, R1.E, R8.2; no longer C27.+, IC5.FB, JP4.10, JP4.12, JP4.2, JP4.4, JP4.6, JP4.8, R27.E, R7.2
- net GND: now also C26.2, C27.2, C28.-, C29.-, C32.2, C34.-, C35.2, D3.A, IC1P.V-, IC4.GND, IC4.OFF, JP4.1, R1.A, R2.2, R20.2, R26.A, R3.1, R4.2, R5.1; no longer C26.-, C27.-, C28.2, C29.2, C32.-, C34.2, D1.A, IC1A.V-, IC6.GND, IC6.OFF, JP3.1, R1.2, R19.2, R2.1, R24.A, R27.A, R3.2, R4.1
- net LCD_A: now also D1.C, R8.1; no longer D3.C, R7.1
- net LCD_CONTR: now also R1.S; no longer R27.S
- net LCD_K: now also D1.A; no longer D3.A
- net LCD_PWM: now also R19.2; no longer R18.2
- net LED_0: now also R27.1; no longer R26.1
- net LED_1: now also R29.1; no longer R28.1
- net LED_2: now also R31.1; no longer R29.1
- net LED_3: now also R33.1; no longer R30.1
- net LED_4: now also R35.1; no longer R31.1
- net LED_5: now also R37.1; no longer R32.1
- net L_FAN_OK: now also R23.2; no longer R22.2
- net N$1: now also D2.C, IC4.OUT; no longer D1.C, IC5.OUT
- net N$10: now also R9.2; no longer R8.2
- net N$11: now also R22.2; no longer R21.2
- net N$12: now also R13.1, R9.1; no longer R12.1, R8.1
- net N$14: now also R10.2; no longer R9.2
- net N$15: now also R2.1, R6.2; no longer R1.1, R5.2
- net N$16: now also R5.2, R7.1; no longer R4.2, R6.1
- net N$17: now also R10.1, R14.1; no longer R13.1, R9.1
- net N$18: now also R15.1; no longer R14.1
- net N$19: now also R4.1, R7.2; no longer R3.1, R6.2
- net N$2: now also R20.1; no longer R18.1
- net N$20: now also R3.2, R6.1; no longer R2.2, R5.1
- net N$21: now also R15.2; no longer R14.2
- net N$22: now also R16.1; no longer R15.1
- net N$23: now also R16.2; no longer R15.2
- net N$24: now also C30.1; no longer C28.1
- net N$25: now also C32.1; no longer C29.1
- net N$26: now also R12.1, R18.2; no longer R11.1, R17.2
- net N$27: now also R11.1, R17.2; no longer R10.1, R16.2
- net N$28: now also R27.2; no longer R26.2
- net N$29: now also R28.1; no longer R33.1
- net N$3: now also D3.C, IC5.OUT; no longer D2.C, IC6.OUT
- net N$30: now also JP3.1, R28.2; no longer JP4.1, R33.2
- net N$31: now also JP3.3, R30.2; no longer JP4.3, R34.2
- net N$32: now also R29.2; no longer R28.2
- net N$33: now also R30.1; no longer R34.1
- net N$34: now also JP3.5, R32.2; no longer JP4.5, R35.2
- net N$35: now also R31.2; no longer R29.2
- net N$36: now also R32.1; no longer R35.1
- net N$37: now also JP3.7, R34.2; no longer JP4.7, R36.2
- net N$38: now also R33.2; no longer R30.2
- net N$39: now also R34.1; no longer R36.1
- net N$40: now also JP3.9, R36.2; no longer JP4.9, R37.2
- net N$41: now also R35.2; no longer R31.2
- net N$42: now also R36.1; no longer R37.1
- net N$43: now also JP3.11; no longer JP4.11
- net N$44: now also R37.2; no longer R32.2
- net N$9: now also R21.2; no longer R20.2
- net NRST: now also JP4.2; no longer JP3.2
- net PWM_FAN_L: now also R21.1, U1.P$60; no longer R20.1
- net PWM_FAN_R: now also R22.1, U1.P$61; no longer R21.1
- net R_FAN_OK: now also R24.2; no longer R23.2
- net SWCLK: now also JP4.3; no longer JP3.3
- net SWDIO: now also JP4.4; no longer JP3.4
- net TACHO_FAN_L: now also R11.2; no longer R10.2
- net TACHO_FAN_R: now also R12.2; no longer R11.2
- net TAMPER: now also C35.1
- net V_DN: now also R26.S; no longer R25.S
- net V_UP: now also R25.S; no longer R24.S
Other:
- moved on the sheet: C30, C31, C33, D2, IC5, R10, R11, R12, R13, R14, R15, R16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

Commit message: Add files via upload
Parts:
- JP1: value (none) -> FAN_R
- JP2: value (none) -> FAN_L
- L7, L8: value (none) -> BEAD
- R1, R25, R26: value (none) -> 10k
- X1: value (none) -> SUPPLY
Connections:
- net PWM_FAN_L: now also R22.1; no longer R21.1
- net PWM_FAN_R: now also R21.1; no longer R22.1
Changed lines of the file:
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@@
 <part name="+3V33" library="supply1" deviceset="+3V3" device=""/>
 <part name="GND30" library="supply1" deviceset="GND" device=""/>
-<part name="X1" library="con-ptr500" deviceset="AK500/2" device=""/>
+<part name="X1" library="con-ptr500" deviceset="AK500/2" device="" value="SUPPLY"/>
 <part name="GND47" library="supply1" deviceset="GND" device=""/>
 <part name="SV1" library="con-harting-ml" deviceset="ML26" device="" value="FRONT_LCD"/>
@@
 <part name="GND44" library="supply1" deviceset="GND" device=""/>
 <part name="+3V312" library="supply1" deviceset="+3V3" device=""/>
-<part name="L7" library="inductor-neosid" deviceset="SM-B" device="5"/>
-<part name="L8" library="inductor-neosid" deviceset="SM-B" device="5"/>
+<part name="L7" library="inductor-neosid" deviceset="SM-B" device="5" value="BEAD"/>
+<part name="L8" library="inductor-neosid" deviceset="SM-B" device="5" value="BEAD"/>
 <part name="C22" library="rcl" deviceset="C-EU" device="C0805" value="100n"/>
 <part name="C23" library="rcl" deviceset="C-EU" device="C0805" value="100n"/>
@@
 <part name="OS1" library="IQD-Frequency-Products" deviceset="OSC-OE" device="-CFPS-39" value="ECS-3225MV-160-CN-TR"/>
 <part name="+3V313" library="supply1" deviceset="+3V3" device=""/>
-<part name="JP1" library="pinhead" deviceset="PINHD-1X3" device=""/>
-<part name="JP2" library="pinhead" deviceset="PINHD-1X3" device=""/>
+<part name="JP1" library="pinhead" deviceset="PINHD-1X3" device="" value="FAN_R"/>
+<part name="JP2" library="pinhead" deviceset="PINHD-1X3" device="" value="FAN_L"/>
 <part name="GND3" library="supply1" deviceset="GND" device=""/>
 <part name="GND4" library="supply1" deviceset="GND" device=""/>
@@
 <part name="R17" library="resistor" deviceset="R-EU_" device="R0805" value="2k7"/>
 <part name="+3V34" library="supply1" deviceset="+3V3" device=""/>
-<part name="R26" library="rcl" deviceset="R-TRIMM" device="3296W"/>
-<part name="R25" library="rcl" deviceset="R-TRIMM" device="3296W"/>
+<part name="R26" library="rcl" deviceset="R-TRIMM" device="3296W" value="10k"/>
+<part name="R25" library="rcl" deviceset="R-TRIMM" device="3296W" value="10k"/>
 <part name="+3V32" library="supply1" deviceset="+3V3" device=""/>
 <part name="GND17" library="supply1" deviceset="GND" device=""/>
@@
 <part name="GND8" library="supply1" deviceset="GND" device=""/>
 <part name="P+2" library="supply1" deviceset="+5V" device=""/>
-<part name="R1" library="pot" deviceset="TRIM_EU-" device="CA6V"/>
+<part name="R1" library="pot" deviceset="TRIM_EU-" device="CA6V" value="10k"/>
 <part name="D1" library="diode" deviceset="1N4148" device="DO35-7" value="1N4148"/>
 <part name="C34" library="rcl" deviceset="CPOL-EU" device="E2-5" value="22u/25"/>
 <part name="P+12" library="supply1" deviceset="+12V" device=""/>
-<part name="GND77" library="supply1" deviceset="GND" device=""/>
+<part name="GND78" library="supply1" deviceset="GND" device=""/>
 <part name="T3" library="transistor" deviceset="BC847" device=""/>
 <part name="R27" library="resistor" deviceset="R-EU_" device="R0805" value="4k7"/>
@@
 <part name="GND54" library="supply1" deviceset="GND" device=""/>
 <part name="IC1" library="linear" deviceset="LM358" device="N"/>
+<part name="GND77" library="supply1" deviceset="GND" device=""/>
 <part name="C35" library="rcl" deviceset="C-EU" device="C0805" value="100n"/>
-<part name="GND78" library="supply1" deviceset="GND" device=""/>
 </parts>
 <sheets>
@@
 <instance part="C34" gate="G$1" x="454.66" y="198.12"/>
 <instance part="P+12" gate="1" x="454.66" y="213.36"/>
-<instance part="GND77" gate="1" x="454.66" y="182.88"/>
+<instance part="GND78" gate="1" x="454.66" y="182.88"/>
 <instance part="T3" gate="G$1" x="274.32" y="-114.3" smashed="yes">
 <attribute name="NAME" x="269.24" y="-109.22" size="1.778" layer="95"/>
@@
 <instance part="IC1" gate="B" x="99.06" y="-10.16" rot="MR0"/>
 <instance part="IC1" gate="P" x="99.06" y="68.58"/>
+<instance part="GND77" gate="1" x="449.58" y="-101.6" rot="R90"/>
 <instance part="C35" gate="G$1" x="441.96" y="-101.6" rot="R90"/>
-<instance part="GND78" gate="1" x="449.58" y="-101.6" rot="R90"/>
 </instances>
 <busses>
@@
 <segment>
 <pinref part="C34" gate="G$1" pin="-"/>
-<pinref part="GND77" gate="1" pin="GND"/>
+<pinref part="GND78" gate="1" pin="GND"/>
 <wire x1="454.66" y1="185.42" x2="454.66" y2="193.04" width="0.1524" layer="91"/>
 </segment>
@@
 </segment>
 <segment>
+<pinref part="GND77" gate="1" pin="GND"/>
 <pinref part="C35" gate="G$1" pin="2"/>
-<pinref part="GND78" gate="1" pin="GND"/>
 </segment>
 </net>
@@
 <net name="PWM_FAN_L" class="0">
 <segment>
-<pinref part="R21" gate="G$1" pin="1"/>
-<wire x1="132.08" y1="71.12" x2="129.54" y2="71.12" width="0.1524" layer="91"/>
-<label x="132.08" y="71.12" size="1.27" layer="95" xref="yes"/>
-</segment>
-<segment>
 <pinref part="U1" gate="G$1" pin="P$60"/>
 <wire x1="424.18" y1="53.34" x2="431.8" y2="53.34" width="0.1524" layer="91"/>
 <label x="431.8" y="53.34" size="1.27" layer="95" xref="yes"/>
+</segment>
+<segment>
+<pinref part="R22" gate="G$1" pin="1"/>
+<wire x1="129.54" y1="-7.62" x2="132.08" y2="-7.62" width="0.1524" layer="91"/>
+<label x="132.08" y="-7.62" size="1.27" layer="95" xref="yes"/>
 </segment>
 </net>
@@
 <net name="PWM_FAN_R" class="0">
 <segment>
-<pinref part="R22" gate="G$1" pin="1"/>
-<wire x1="132.08" y1="-7.62" x2="129.54" y2="-7.62" width="0.1524" layer="91"/>
-<label x="132.08" y="-7.62" size="1.27" layer="95" xref="yes"/>
-</segment>
-<segment>
 <pinref part="U1" gate="G$1" pin="P$61"/>
 <wire x1="424.18" y1="55.88" x2="431.8" y2="55.88" width="0.1524" layer="91"/>
 <label x="431.8" y="55.88" size="1.27" layer="95" xref="yes"/>
+</segment>
+<segment>
+<pinref part="R21" gate="G$1" pin="1"/>
+<wire x1="129.54" y1="71.12" x2="132.08" y2="71.12" width="0.1524" layer="91"/>
+<label x="132.08" y="71.12" size="1.27" layer="95" xref="yes"/>
 </segment>
 </net>
@@
 <junction x="436.88" y="-106.68"/>
 <label x="444.5" y="-106.68" size="1.27" layer="95" xref="yes"/>
-<pinref part="C35" gate="G$1" pin="1"/>
 <wire x1="439.42" y1="-101.6" x2="436.88" y2="-101.6" width="0.1524" layer="91"/>
 <junction x="436.88" y="-101.6"/>
-</segment>
-</net>
+<pinref part="C35" gate="G$1" pin="1"/>
+</segment>
+</net>

Commit message: Add files via upload
Parts:
- added C36: 22u/25, rcl:CPOL-EUE2-5
- added C37, C38: 10n, rcl:C-EUC0805
- added JP7: ENCODER, pinhead:PINHD-1X3
- added R44, R45, R46, R47: 10k, rcl:R-EU_R0805
- added TP1, TP2, TP3, TP4, TP5, TP6, TP7, TP8: TPB2,54, testpad:TPB2,54
- C11: value 1u -> 100u/35V; device rcl:C-EUC0805 -> rcl:CPOL-EUE3.5-8
- C13: value 100n -> 1u
- C20: value 10n -> 100n
- C21: value 100n -> 10n
- C24: value 100u/35V -> 100n; device rcl:CPOL-EUE3.5-8 -> rcl:C-EUC0805
- C26: value 10u/TA -> 100u/35V; device resistor:C-EUC1206 -> rcl:CPOL-EUE3.5-8
- C28: value 1000u/10V -> 10u/TA; device rcl:CPOL-EUE3.5-8 -> resistor:C-EUC1206
- C30: value 2u2 -> 1000u/10V; device rcl:C-EUC0805 -> rcl:CPOL-EUE3.5-8
- C31: value 100n -> 2u2
- C32: value 2u2 -> 100n
- C33: value 4.7u -> 2u2
- C34: value 22u/25 -> 4.7u; device rcl:CPOL-EUE2-5 -> rcl:C-EUC0805
- D1: value 1N4148 -> 1N5822; device diode:1N4148DO35-7 -> diode:1N5819-T
- R8: device resistor:R-EU_R0805 -> rcl:R-EU_R1206
Connections:
- new net N$47: TP7.TP, U1.P$1
- new net N$48: JP7.3, R45.1, R46.1
- new net N$49: JP7.1, R44.1, R47.1
- new net N$50: TP8.TP, U1.P$2
- net +12V: now also C11.+, C26.+, C36.+, TP1.TP; no longer C24.+, C34.+
- net +3V3: now also C14.1, C22.1, C28.1, C29.+, C32.1, C34.1, R46.2, R47.2, TP2.TP; no longer C13.1, C20.1, C26.1, C28.+, C31.1, C33.1
- net +5V: now also C18.2, C30.+, TP3.TP; no longer C17.2, C29.+
- net 32M_REF_OUT: now also TP6.TP
- net ENC_A: now also C38.1, R45.2
- net ENC_B: now also C37.1, R44.2
- net GND: now also C11.-, C17.2, C20.1, C24.2, C26.-, C28.2, C30.-, C34.2, C36.-, C37.2, C38.2, JP7.2; no longer C11.2, C17.1, C20.2, C24.-, C26.2, C28.-, C30.2, C34.-
- net N$11: now also C13.1; no longer C12.1
- net N$15: now also TP5.TP
- net N$19: now also TP4.TP
- net N$24: now also C31.1; no longer C30.1
- net N$25: now also C33.1; no longer C32.1
- net N$4: now also C15.1; no longer C14.1
- net N$5: now also C19.2; no longer C18.2
- net N$6: now also C20.2; no longer C19.2
- net N$9: now also C12.1; no longer C11.1
- net VDDA: now also C23.1; no longer C22.1
- net VREF: now also C24.1; no longer C23.1
- net V_DN: now also C17.1; no longer C16.1
- net V_UP: now also C16.1; no longer C15.1
Other:
- moved on the sheet: C12, C13, C14, C15, C16, C17, C18, C19, C20, C21, C22, C23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

Commit message: Add files via upload
Connections:
- net GND: now also IC4.TAB, IC5.TAB
- net LCD_CS1: now also U1.P$15
- net LCD_CS2: now also U1.P$16
- net LCD_CS3: now also U1.P$17
Changed lines of the file:
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@@
 <pinref part="IC4" gate="A" pin="OFF"/>
 <wire x1="309.88" y1="238.76" x2="307.34" y2="238.76" width="0.1524" layer="91"/>
-<wire x1="307.34" y1="238.76" x2="307.34" y2="200.66" width="0.1524" layer="91"/>
+<wire x1="307.34" y1="238.76" x2="307.34" y2="233.68" width="0.1524" layer="91"/>
 <pinref part="GND53" gate="1" pin="GND"/>
 <pinref part="IC5" gate="A" pin="OFF"/>
-<wire x1="307.34" y1="200.66" x2="307.34" y2="185.42" width="0.1524" layer="91"/>
+<wire x1="307.34" y1="233.68" x2="307.34" y2="200.66" width="0.1524" layer="91"/>
+<wire x1="307.34" y1="200.66" x2="307.34" y2="195.58" width="0.1524" layer="91"/>
+<wire x1="307.34" y1="195.58" x2="307.34" y2="185.42" width="0.1524" layer="91"/>
 <wire x1="309.88" y1="200.66" x2="307.34" y2="200.66" width="0.1524" layer="91"/>
 <junction x="307.34" y="200.66"/>
+<pinref part="IC4" gate="A" pin="TAB"/>
+<wire x1="309.88" y1="233.68" x2="307.34" y2="233.68" width="0.1524" layer="91"/>
+<pinref part="IC5" gate="A" pin="TAB"/>
+<wire x1="309.88" y1="195.58" x2="307.34" y2="195.58" width="0.1524" layer="91"/>
+<junction x="307.34" y="195.58"/>
+<junction x="307.34" y="233.68"/>
 </segment>
 <segment>
@@
 <label x="45.72" y="243.84" size="1.27" layer="95" xref="yes"/>
 </segment>
+<segment>
+<pinref part="U1" gate="G$1" pin="P$16"/>
+<wire x1="327.66" y1="53.34" x2="317.5" y2="53.34" width="0.1524" layer="91"/>
+<label x="317.5" y="53.34" size="1.27" layer="95" rot="R180" xref="yes"/>
+</segment>
 </net>
 <net name="LCD_RES" class="0">
@@
 <label x="25.4" y="241.3" size="1.27" layer="95" rot="R180" xref="yes"/>
 </segment>
+<segment>
+<pinref part="U1" gate="G$1" pin="P$15"/>
+<wire x1="327.66" y1="55.88" x2="317.5" y2="55.88" width="0.1524" layer="91"/>
+<label x="317.5" y="55.88" size="1.27" layer="95" rot="R180" xref="yes"/>
+</segment>
 </net>
 <net name="LCD_CS3" class="0">
@@
 <label x="25.4" y="243.84" size="1.27" layer="95" rot="R180" xref="yes"/>
 </segment>
-</net>
+<segment>
+<pinref part="U1" gate="G$1" pin="P$17"/>
+<wire x1="327.66" y1="50.8" x2="317.5" y2="50.8" width="0.1524" layer="91"/>
+<label x="317.5" y="50.8" size="1.27" layer="95" rot="R180" xref="yes"/>
+</segment>
+</net>

Commit message: Add files via upload
Parts:
- removed SV6: RESERVED, con-harting-ml:ML10
- added H1, H2, H3, H4, H5, H6: MOUNT-PAD-ROUND3.2, holes:MOUNT-PAD-ROUND3.2
- added R48, R49: 10k, resistor:R-EU_R0805
Connections:
- removed net PTT: U1.P$97
- removed net USART1_RX: U1.P$69
- removed net USART1_TX: U1.P$68
- net +3V3: now also R48.2
- net ANALOG_IN_0: now also SV3.6
- net BTN_0: now also U1.P$88; no longer U1.P$83
- net BTN_1: now also U1.P$85; no longer U1.P$84
- net BTN_2: now also U1.P$84; no longer U1.P$85
- net BTN_3: now also U1.P$83; no longer U1.P$88
- net DAC_OUT: now also SV3.8
- net ENC_A: now also U1.P$90; no longer U1.P$91
- net ENC_B: now also U1.P$91; no longer U1.P$90
- net FRONT_PTT: now also R49.1, U1.P$97
- net FRONT_RX: now also U1.P$69
- net FRONT_TX: now also U1.P$68
- net GND: now also H1.MOUNT, H2.MOUNT, H3.MOUNT, H4.MOUNT, H5.MOUNT, H6.MOUNT
- net LED_0: now also R37.1; no longer R27.1
- net LED_1: now also R35.1; no longer R29.1
- net LED_2: now also R33.1; no longer R31.1
- net LED_3: now also R31.1; no longer R33.1
- net LED_4: now also R29.1; no longer R35.1
- net LED_5: now also R27.1; no longer R37.1
- net N$13: now also R49.2
- net NRST: now also R48.1

Commit message: Add files via upload
Parts:
- removed TP6: TPB2,54, testpad:TPB2,54
Connections:
- net 32M_REF_OUT: no longer TP6.TP
Changed lines of the file:
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@@
 <part name="TP4" library="testpad" deviceset="TP" device="B2,54"/>
 <part name="TP5" library="testpad" deviceset="TP" device="B2,54"/>
-<part name="TP6" library="testpad" deviceset="TP" device="B2,54"/>
 <part name="TP7" library="testpad" deviceset="TP" device="B2,54"/>
 <part name="TP8" library="testpad" deviceset="TP" device="B2,54"/>
@@
 <instance part="TP4" gate="G$1" x="63.5" y="25.4"/>
 <instance part="TP5" gate="G$1" x="63.5" y="104.14"/>
-<instance part="TP6" gate="G$1" x="160.02" y="254"/>
 <instance part="TP7" gate="G$1" x="317.5" y="101.6"/>
 <instance part="TP8" gate="G$1" x="307.34" y="101.6"/>
@@
 <pinref part="IC3" gate="B" pin="I0"/>
 <wire x1="170.18" y1="248.92" x2="165.1" y2="248.92" width="0.1524" layer="91"/>
-<pinref part="TP6" gate="G$1" pin="TP"/>
-<wire x1="160.02" y1="251.46" x2="160.02" y2="248.92" width="0.1524" layer="91"/>
-<wire x1="160.02" y1="248.92" x2="165.1" y2="248.92" width="0.1524" layer="91"/>
-<junction x="165.1" y="248.92"/>
 </segment>
 </net>
