File: schematics/mainboard/mainboard.sch (EAGLE design)
At the start: 144 parts, among them IC1 LM358N, IC2 LM339N, IC3 74AHC00D, IC4 LM2576-5.0, IC5 LM2576-3.3, Q1 BD140, Q2 BD140, Q3 IRF540, T1 2N3904, T2 2N3904, T3 BC847, T4 BC847, T5 BC847, T6 BC847, T7 BC847, T8 BC847, U1 STM32F777VIT, X1 SUPPLY

Commit message: Add files via upload
Parts:
- L10, L9: value 100u/5A -> 1410454C
- Q3: value IRF540 -> IRL520
Connections:
- net +12V: now also C34.1, IC2P.V+
- net +3V3: no longer C34.1, IC2P.V+
- net N$26: now also IC2C.-IN; no longer IC2C.+IN
- net V_UP: now also IC2C.+IN; no longer IC2C.-IN
Other:
- moved on the sheet: IC2C
Changed lines of the file:
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@@
 <part name="IC5" library="v-reg-3" deviceset="LM2576" device="S" value="LM2576-3.3"/>
 <part name="D3" library="diode" deviceset="1N581*" device="" technology="9-T" value="1N5822"/>
-<part name="L10" library="rcl" deviceset="L-EU" device="TJ5-U2" value="100u/5A"/>
-<part name="L9" library="rcl" deviceset="L-EU" device="TJ5-U2" value="100u/5A"/>
+<part name="L10" library="rcl" deviceset="L-EU" device="TJ5-U2" value="1410454C"/>
+<part name="L9" library="rcl" deviceset="L-EU" device="TJ5-U2" value="1410454C"/>
 <part name="GND59" library="supply1" deviceset="GND" device=""/>
 <part name="GND61" library="supply1" deviceset="GND" device=""/>
@@
 <part name="GND2" library="supply1" deviceset="GND" device=""/>
 <part name="GND1" library="supply1" deviceset="GND" device=""/>
-<part name="Q3" library="transistor-power" deviceset="IRF540" device=""/>
+<part name="Q3" library="transistor-power" deviceset="IRF540" device="" value="IRL520"/>
 <part name="GND13" library="supply1" deviceset="GND" device=""/>
 <part name="GND20" library="supply1" deviceset="GND" device=""/>
@@
 <part name="GND35" library="supply1" deviceset="GND" device=""/>
 <part name="GND75" library="supply1" deviceset="GND" device=""/>
-<part name="+3V326" library="supply1" deviceset="+3V3" device=""/>
 <part name="C34" library="rcl" deviceset="C-EU" device="C0805" value="4.7u"/>
 <part name="GND42" library="supply1" deviceset="GND" device=""/>
@@
 <part name="GND83" library="supply1" deviceset="GND" device=""/>
 <part name="H6" library="holes" deviceset="MOUNT-PAD-ROUND" device="3.2"/>
+<part name="P+14" library="supply1" deviceset="+12V" device=""/>
 </parts>
 <sheets>
@@
 <instance part="IC2" gate="A" x="124.46" y="-88.9" rot="MR180"/>
 <instance part="IC2" gate="B" x="124.46" y="-109.22"/>
-<instance part="IC2" gate="C" x="124.46" y="-139.7"/>
+<instance part="IC2" gate="C" x="124.46" y="-139.7" rot="MR180"/>
 <instance part="IC2" gate="D" x="124.46" y="-160.02"/>
 <instance part="R11" gate="G$1" x="76.2" y="-86.36" rot="R180"/>
@@
 <instance part="GND35" gate="1" x="177.8" y="-114.3"/>
 <instance part="GND75" gate="1" x="431.8" y="182.88"/>
-<instance part="+3V326" gate="G$1" x="431.8" y="213.36"/>
 <instance part="C34" gate="G$1" x="441.96" y="198.12"/>
 <instance part="GND42" gate="1" x="223.52" y="101.6"/>
@@
 <instance part="GND83" gate="1" x="185.42" y="27.94"/>
 <instance part="H6" gate="G$1" x="236.22" y="38.1" rot="R90"/>
+<instance part="P+14" gate="1" x="431.8" y="213.36"/>
 </instances>
 <busses>
@@
 <pinref part="R26" gate="G$1" pin="E"/>
 <pinref part="+3V39" gate="G$1" pin="+3V3"/>
-</segment>
-<segment>
-<pinref part="+3V326" gate="G$1" pin="+3V3"/>
-<wire x1="431.8" y1="210.82" x2="431.8" y2="208.28" width="0.1524" layer="91"/>
-<pinref part="C34" gate="G$1" pin="1"/>
-<wire x1="431.8" y1="208.28" x2="431.8" y2="205.74" width="0.1524" layer="91"/>
-<wire x1="441.96" y1="200.66" x2="441.96" y2="208.28" width="0.1524" layer="91"/>
-<wire x1="441.96" y1="208.28" x2="431.8" y2="208.28" width="0.1524" layer="91"/>
-<junction x="431.8" y="208.28"/>
-<pinref part="IC2" gate="P" pin="V+"/>
 </segment>
 <segment>
@@
 <wire x1="114.3" y1="91.44" x2="111.76" y2="91.44" width="0.1524" layer="91"/>
 </segment>
+<segment>
+<pinref part="C34" gate="G$1" pin="1"/>
+<wire x1="431.8" y1="208.28" x2="431.8" y2="205.74" width="0.1524" layer="91"/>
+<wire x1="441.96" y1="200.66" x2="441.96" y2="208.28" width="0.1524" layer="91"/>
+<wire x1="441.96" y1="208.28" x2="431.8" y2="208.28" width="0.1524" layer="91"/>
+<pinref part="IC2" gate="P" pin="V+"/>
+<pinref part="P+14" gate="1" pin="+12V"/>
+<wire x1="431.8" y1="210.82" x2="431.8" y2="208.28" width="0.1524" layer="91"/>
+<junction x="431.8" y="208.28"/>
+</segment>
 </net>
 <net name="N$1" class="0">
@@
 </segment>
 <segment>
-<wire x1="116.84" y1="-142.24" x2="106.68" y2="-142.24" width="0.1524" layer="91"/>
-<label x="106.68" y="-142.24" size="1.27" layer="95" rot="R180" xref="yes"/>
-<pinref part="IC2" gate="C" pin="-IN"/>
-</segment>
-<segment>
 <pinref part="R25" gate="G$1" pin="S"/>
 <pinref part="C16" gate="G$1" pin="1"/>
@@
 <label x="180.34" y="-101.6" size="1.27" layer="95" xref="yes"/>
 </segment>
+<segment>
+<pinref part="IC2" gate="C" pin="+IN"/>
+<wire x1="116.84" y1="-142.24" x2="106.68" y2="-142.24" width="0.1524" layer="91"/>
+<label x="106.68" y="-142.24" size="1.27" layer="95" rot="R180" xref="yes"/>
+</segment>
 </net>
 <net name="V_DN" class="0">
@@
 <wire x1="116.84" y1="-111.76" x2="106.68" y2="-111.76" width="0.1524" layer="91"/>
 <label x="106.68" y="-111.76" size="1.27" layer="95" rot="R180" xref="yes"/>
-</segment>
-<segment>
-<wire x1="116.84" y1="-162.56" x2="106.68" y2="-162.56" width="0.1524" layer="91"/>
-<label x="106.68" y="-162.56" size="1.27" layer="95" rot="R180" xref="yes"/>
-<pinref part="IC2" gate="D" pin="-IN"/>
 </segment>
 <segment>
@@
 <label x="180.34" y="-121.92" size="1.27" layer="95" xref="yes"/>
 </segment>
+<segment>
+<pinref part="IC2" gate="D" pin="-IN"/>
+<wire x1="116.84" y1="-162.56" x2="106.68" y2="-162.56" width="0.1524" layer="91"/>
+<label x="106.68" y="-162.56" size="1.27" layer="95" rot="R180" xref="yes"/>
+</segment>
 </net>
 <net name="N$26" class="0">
@@
 <pinref part="C6" gate="G$1" pin="+"/>
 <wire x1="83.82" y1="-137.16" x2="83.82" y2="-139.7" width="0.1524" layer="91"/>
-<wire x1="83.82" y1="-137.16" x2="111.76" y2="-137.16" width="0.1524" layer="91"/>
-<wire x1="111.76" y1="-137.16" x2="116.84" y2="-137.16" width="0.1524" layer="91"/>
-<wire x1="116.84" y1="-157.48" x2="111.76" y2="-157.48" width="0.1524" layer="91"/>
-<wire x1="111.76" y1="-157.48" x2="111.76" y2="-137.16" width="0.1524" layer="91"/>
 <junction x="83.82" y="-137.16"/>
+<pinref part="IC2" gate="C" pin="-IN"/>
+<wire x1="116.84" y1="-137.16" x2="111.76" y2="-137.16" width="0.1524" layer="91"/>
+<wire x1="111.76" y1="-137.16" x2="83.82" y2="-137.16" width="0.1524" layer="91"/>
+<wire x1="111.76" y1="-137.16" x2="111.76" y2="-157.48" width="0.1524" layer="91"/>
 <junction x="111.76" y="-137.16"/>
-<pinref part="IC2" gate="C" pin="+IN"/>
 <pinref part="IC2" gate="D" pin="+IN"/>
+<wire x1="111.76" y1="-157.48" x2="116.84" y2="-157.48" width="0.1524" layer="91"/>
 </segment>
 </net>
 <net name="R_FAN_OK" class="0">
 <segment>
-<pinref part="IC2" gate="D" pin="OUT"/>
 <pinref part="R24" gate="G$1" pin="2"/>
-<wire x1="132.08" y1="-160.02" x2="137.16" y2="-160.02" width="0.1524" layer="91"/>
 <wire x1="137.16" y1="-160.02" x2="137.16" y2="-139.7" width="0.1524" layer="91"/>
-<pinref part="IC2" gate="C" pin="OUT"/>
 <wire x1="137.16" y1="-139.7" x2="137.16" y2="-134.62" width="0.1524" layer="91"/>
-<wire x1="132.08" y1="-139.7" x2="137.16" y2="-139.7" width="0.1524" layer="91"/>
 <junction x="137.16" y="-139.7"/>
 <wire x1="137.16" y1="-139.7" x2="139.7" y2="-139.7" width="0.1524" layer="91"/>
 <label x="139.7" y="-139.7" size="1.27" layer="95" xref="yes"/>
-</segment>
-</net>
+<pinref part="IC2" gate="C" pin="OUT"/>
+<wire x1="132.08" y1="-139.7" x2="137.16" y2="-139.7" width="0.1524" layer="91"/>
+<pinref part="IC2" gate="D" pin="OUT"/>
+<wire x1="132.08" y1="-160.02" x2="137.16" y2="-160.02" width="0.1524" layer="91"/>
+</segment>
+</net>

Commit message: Add files via upload
Parts:
- removed C11, C25, C26, C3, C4: 100u/35V, rcl:CPOL-EUE3.5-8
- removed C12, C13: 1u, rcl:C-EUC0805
- removed C16, C17: 100n, rcl:C-EUC0805
- removed C34: 4.7u, rcl:C-EUC0805
- removed C36, C5, C6: 22u/25, rcl:CPOL-EUE2-5
- removed D2, D3: 1N5822, diode:1N5819-T
- removed H1, H4: MOUNT-PAD-ROUND3.2, holes:MOUNT-PAD-ROUND3.2
- removed IC1: LM358N, linear:LM358N
- removed IC2: LM339N, linear:LM339N
- removed IC4: LM2576-5.0, v-reg-3:LM2576S
- removed IC5: LM2576-3.3, v-reg-3:LM2576S
- removed JP1: FAN_R, pinhead:PINHD-1X3
- removed JP2: FAN_L, pinhead:PINHD-1X3
- removed L10, L9: 1410454C, rcl:L-EUTJ5-U2
- removed Q1, Q2: BD140, transistor-power:BD140
- removed R10, R9: 470R, resistor:R-EU_R0805
- removed R11, R12, R15, R16, R23, R24: 4k7, resistor:R-EU_R0805
- removed R13, R14, R2, R4: 10k, resistor:R-EU_R0805
- removed R17, R18, R6, R7: 2k7, resistor:R-EU_R0805
- removed R21, R22: 22k, resistor:R-EU_R0805
- removed R25, R26: 10k, rcl:R-TRIMM3296W
- removed R3, R5: 1k, resistor:R-EU_R0805
- removed T1, T2: 2N3904, transistor-neu-to92:2N3904-NPN-TO92-EBC
- removed TP1, TP2, TP3, TP4, TP5: TPB2,54, testpad:TPB2,54
- removed X1: SUPPLY, con-ptr500:AK500/2
- added X2: (no value), con-ptr500:AK500/4
- D1: value 1N5822 -> UF4007
Connections:
- removed net +12V: C11.+, C25.+, C26.+, C34.1, C36.+, IC1P.V+, IC2P.V+, IC4.VIN, IC5.VIN, Q1.E, Q2.E, R13.2, R14.2, TP1.TP, X1-1.KL
- removed net L_FAN_OK: IC2A.OUT, IC2B.OUT, R23.2
- removed net N$1: D2.C, IC4.OUT, L10.1
- removed net N$10: R9.2, T1.C
- removed net N$11: C13.1, IC1B.+IN, R22.2
- removed net N$12: Q1.B, R13.1, R9.1
- removed net N$14: R10.2, T2.C
- removed net N$15: C3.+, JP1.1, Q1.C, R2.1, R6.2, TP5.TP
- removed net N$16: IC1B.-IN, R5.2, R7.1
- removed net N$17: Q2.B, R10.1, R14.1
- removed net N$18: R15.1, T1.B
- removed net N$19: C4.+, JP2.1, Q2.C, R4.1, R7.2, TP4.TP
- removed net N$20: IC1A.-IN, R3.2, R6.1
- removed net N$21: IC1A.OUT, R15.2
- removed net N$22: R16.1, T2.B
- removed net N$23: IC1B.OUT, R16.2
- removed net N$26: C6.+, IC2C.-IN, IC2D.+IN, R12.1, R18.2
- removed net N$27: C5.+, IC2A.-IN, IC2B.+IN, R11.1, R17.2
- removed net N$3: D3.C, IC5.OUT, L9.1
- removed net N$9: C12.1, IC1A.+IN, R21.2
- removed net R_FAN_OK: IC2C.OUT, IC2D.OUT, R24.2
- removed net TACHO_FAN_L: JP2.2, R11.2
- removed net TACHO_FAN_R: JP1.2, R12.2
- removed net V_DN: C17.1, IC2B.-IN, IC2D.-IN, R26.S
- removed net V_UP: C16.1, IC2A.+IN, IC2C.+IN, R25.S
- net +3V3: now also X2-2.KL; no longer IC5.FB, L9.2, R17.1, R18.1, R23.1, R24.1, R25.E, R26.E, TP2.TP
- net +5V: now also X2-1.KL; no longer IC4.FB, L10.2, TP3.TP
- net GND: now also X2-3.KL, X2-4.KL; no longer C11.-, C12.2, C13.2, C16.2, C17.2, C25.-, C26.-, C3.-, C34.2, C36.-, C4.-, C5.-, C6.-, D2.A, D3.A, H1.MOUNT, H4.MOUNT, IC1P.V-, IC2P.GND, IC4.GND, IC4.OFF, IC4.TAB, IC5.GND, IC5.OFF, IC5.TAB, JP1.3, JP2.3, R2.2, R25.A, R26.A, R3.1, R4.2, R5.1, T1.E, T2.E, X1-2.KL
- net PWM_FAN_L: no longer R22.1
- net PWM_FAN_R: no longer R21.1
Other:
- note removed: "SHIELDED"
- moved on the sheet: C29, C30, C32, H2, H3, H5, H6, IC3P
