File: schematics/fan_ctrl/fan_ctrl.sch (EAGLE design)
At the start: 48 parts, among them IC1 LD117AS50TR, IC2 74HC590N, IC3 74HC590N, IC4 74HC590N, IC5 PCF8574P, IC6 PCF8574P, IC7 LM358N, Q1 BSS123, Q2 BSS123, Q3 BD140, Q4 BD140, T1 2N3904, T2 2N3904

Commit message: Add files via upload
Parts:
- added C10, C11, C12, C13, C9: 1u, rcl:C-EUC0805
- added H1, H2, H3, H4: MOUNT-PAD-ROUND3.2, holes:MOUNT-PAD-ROUND3.2
- added TP4: TPB2,54, testpad:TPB2,54
Connections:
- net +5V: now also C10.1, C11.1, C12.1, C13.1, C9.1, IC2P.VCC, IC3P.VCC, IC4P.VCC
- net FAN_L: now also IC5.P7; no longer IC5.P6
- net FAN_R: now also IC5.P6; no longer IC5.P7
- net GND: now also C10.2, C11.2, C12.2, C13.2, C9.2, H1.MOUNT, H2.MOUNT, H3.MOUNT, H4.MOUNT, IC2P.GND, IC3P.GND, IC4P.GND
- net N$7: now also TP4.TP
- net PWM_FAN_L: now also JP3.2; no longer JP3.3
- net PWM_FAN_R: now also JP3.3; no longer JP3.2
Other:
- moved on the sheet: C1, C2, IC1
