File: schematics/supply_board/supply_board.sch (EAGLE design)
At the start: 68 parts, among them IC1 HLSR_10-P, IC2 LM324N, IC3 AIMTEC 5.0V, IC4 AIMTEC 3.3V, IC5 LD117AS50TR, IC6 MCP3208, IC7 AD7524JN, IC8 PCF8574P, Q1 TIP36C, Q2 BD139-16, Q3 TIP36C, Q4 BD139-16, U1 VOLT_REFERENCE

Commit message: Add files via upload
Parts:
- removed IC5: LD117AS50TR, v-reg:LD117AS50TR
- added C20: ?, rcl:CPOL-EUE5-13
- added C21: 1u, rcl:C-EUC0805
- added C22: (no value), rcl:CPOL-EUE2.5-6
- added IC10: LM340S, linear:LM340S
- added IC9: AIMTEC 5.0V, linear:7805TV
- added JP5: (no value), pinhead:PINHD-1X8
- added R20: 18k, resistor:R-EU_R0805
- added R21: 1k, resistor:R-EU_R0805
- added X7: (no value), con-ptr500:AK500/2
- D2: value 1N4004 -> BZX85-3V3; device diode:1N4004 -> diode:BZX85
- R16: value 47R/3W -> 2k; device rcl:R-EU_0411/15 -> resistor:R-EU_R0805
- R6: device rcl:R-EU_0411/15 -> rcl:R-EU_0617/22
Connections:
- removed net N$28: D2.A, Q4.E
- new net 5V_OUT_B: C21.1, C22.+, IC9.VO, JP5.1, JP5.2, JP5.3, JP5.4, JP5.5, JP5.6, JP5.7, JP5.8
- new net N$24: D2.C, Q4.E
- net +15V: now also IC10.IN, IC9.VI; no longer IC5.IN
- net +5V: now also IC10.OUT; no longer IC5.OUT
- net 12V_OUT: now also C20.+, X7-2.KL
- net GND: now also C20.-, C21.2, C22.-, D2.A, IC10.GND@1, IC7.OUT1, IC9.GND, R16.2, R20.1, X7-1.KL; no longer D2.C, IC5.ADJ, IC7.OUT2
- net I_REF: now also IC7.OUT2; no longer IC7.OUT1
- net MISO: now also R21.2; no longer JP1.4
- net N$12: now also R20.2
- net N$18: now also Q4.C; no longer R16.2
- net N$27: now also JP1.4, R21.1; no longer Q4.C
Other:
- moved on the sheet: C16, C19, C7, JP1, R16, X5-1, X5-2, X6-1, X6-2

Commit message: Add files via upload
Parts:
- removed IC9: AIMTEC 5.0V, linear:7805TV
- added C23: 1000u/25V, rcl:CPOL-EUE5-10.5
- added D3: 1N5822, diode:1N5908
- added IC5: LM2576S, v-reg-3:LM2576S
- added L1: 100u/5A, rcl:L-EUTJ5-U2
- added R22: 47R, resistor:R-EU_R0805
- C21: value 1u -> 100u/35V; device rcl:C-EUC0805 -> rcl:CPOL-EUE5-10.5
Connections:
- new net N$31: IC5.FB, R22.2
- new net N$33: D3.C, IC5.OUT, L1.1
- net +15V: now also C21.+, IC5.VIN; no longer IC9.VI
- net 5V_OUT_B: now also C23.+, L1.2, R22.1; no longer C21.1, IC9.VO
- net GND: now also C21.-, C23.-, D3.A, IC5.GND, IC5.OFF, IC5.TAB; no longer C21.2, IC9.GND

Commit message: Add files via upload
Other:
- moved on the sheet: R17, R18
Changed lines of the file:
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@@
 <instance part="GND39" gate="1" x="248.92" y="177.8"/>
 <instance part="GND40" gate="1" x="269.24" y="177.8"/>
-<instance part="R17" gate="G$1" x="284.48" y="182.88" rot="R180"/>
-<instance part="R18" gate="G$1" x="294.64" y="182.88" rot="R180"/>
+<instance part="R17" gate="G$1" x="284.48" y="190.5" rot="R180"/>
+<instance part="R18" gate="G$1" x="294.64" y="190.5" rot="R180"/>
 <instance part="GND41" gate="1" x="302.26" y="177.8"/>
 <instance part="R19" gate="G$1" x="276.86" y="200.66" rot="R90"/>
@@
 <pinref part="R18" gate="G$1" pin="1"/>
 <pinref part="GND41" gate="1" pin="GND"/>
-<wire x1="299.72" y1="182.88" x2="302.26" y2="182.88" width="0.1524" layer="91"/>
-<wire x1="302.26" y1="182.88" x2="302.26" y2="180.34" width="0.1524" layer="91"/>
+<wire x1="299.72" y1="190.5" x2="302.26" y2="190.5" width="0.1524" layer="91"/>
+<wire x1="302.26" y1="190.5" x2="302.26" y2="180.34" width="0.1524" layer="91"/>
 </segment>
 <segment>
@@
 <segment>
 <pinref part="R19" gate="G$1" pin="1"/>
-<wire x1="276.86" y1="195.58" x2="276.86" y2="182.88" width="0.1524" layer="91"/>
+<wire x1="276.86" y1="195.58" x2="276.86" y2="190.5" width="0.1524" layer="91"/>
+<pinref part="R17" gate="G$1" pin="2"/>
+<wire x1="276.86" y1="190.5" x2="279.4" y2="190.5" width="0.1524" layer="91"/>
 <pinref part="VR1" gate="G$1" pin="R"/>
-<wire x1="276.86" y1="182.88" x2="274.32" y2="187.96" width="0.1524" layer="91"/>
-<pinref part="R17" gate="G$1" pin="2"/>
-<wire x1="276.86" y1="182.88" x2="279.4" y2="182.88" width="0.1524" layer="91"/>
-<junction x="276.86" y="182.88"/>
-</segment>
-</net>
+<wire x1="276.86" y1="190.5" x2="274.32" y2="190.5" width="0.1524" layer="91"/>
+<wire x1="274.32" y1="190.5" x2="274.32" y2="187.96" width="0.1524" layer="91"/>
+<junction x="276.86" y="190.5"/>
+</segment>
+</net>

Commit message: Add files via upload
Parts:
- removed C17: (no value), rcl:CPOL-EUE2.5-6
- removed JP2: (no value), pinhead:PINHD-2X8
- removed X5: (no value), con-ptr500:AK500/2
- added C24: 1u, rcl:C-EUC0805
- added JP6, JP7, JP8: (no value), pinhead:PINHD-1X8
Connections:
- net 5V_OUT: no longer C17.+, X5-2.KL
- net 5V_OUT_B: now also C24.2
- net GND: now also C24.1, JP6.1, JP6.2, JP6.3, JP6.4, JP6.5, JP6.6, JP6.7, JP6.8, JP7.1, JP7.2, JP7.3, JP7.4, JP7.5, JP7.6, JP7.7, JP7.8, JP8.1, JP8.2, JP8.3, JP8.4, JP8.5, JP8.6, JP8.7, JP8.8; no longer C17.-, JP2.1, JP2.10, JP2.11, JP2.12, JP2.13, JP2.14, JP2.15, JP2.16, JP2.2, JP2.3, JP2.4, JP2.5, JP2.6, JP2.7, JP2.8, JP2.9, X5-1.KL
Other:
- moved on the sheet: C16
