File: schematics/supply_board/supply_board.brd (EAGLE design)
At the start: 163 x 99 mm, 68 parts, among them IC1 HLSR_10-P, IC2 LM324N, IC3 AIMTEC 5.0V, IC4 AIMTEC 3.3V, IC5 LD117AS50TR, IC6 MCP3208, IC7 AD7524JN, IC8 PCF8574P, Q1 TIP36C, Q2 BD139-16, Q3 TIP36C, Q4 BD139-16, U1 VOLT_REFERENCE

Commit message: Add files via upload
Parts:
- added C20: ?, rcl:E5-13
- added C21: 100u/35V, rcl:E5-10,5
- added C22: (no value), rcl:E2,5-6
- added C23: 1000u/25V, rcl:E5-10,5
- added D3: 1N5822, diode:C4111-15
- added IC10: LM340S, linear:SOT223
- added JP5: (no value), pinhead:1X08
- added L1: 100u/5A, rcl:TJ5-U2
- added R20: 18k, resistor:R0805
- added R21: 1k, resistor:R0805
- added R22: 47R, resistor:R0805
- added X7: (no value), con-ptr500:AK500/2
- D2: value 1N4004 -> BZX85-3V3; device diode:DO41-10 -> diode:DO41Z10
- IC5: value LD117AS50TR -> LM2576S; device v-reg:SOT223 -> v-reg-3:TO263-5
- R16: value 47R/3W -> 2k; device rcl:0411/15 -> resistor:R0805
- R6: device rcl:0411/15 -> rcl:0617/22
- moved R16 179.9 mm to (-21.6, -94.6), turned to 0 degrees
- moved IC5 146.4 mm to (8.26, -85.1), turned to 0 degrees
- moved D2 0.36 mm to (22.0, 81.0), turned to 90 degrees
Connections:
- removed net N$28: D2.A, Q4.E
- new net 5V_OUT_B: C22.+, C23.+, JP5.1, JP5.2, JP5.3, JP5.4, JP5.5, JP5.6, JP5.7, JP5.8, L1.2, R22.1
- new net N$24: D2.C, Q4.E
- new net N$31: IC5.4, R22.2
- new net N$33: D3.C, IC5.2, L1.1
- net +15V: now also C21.+, IC10.1, IC5.1; no longer IC5.3
- net +5V: now also IC10.3; no longer IC5.4
- net 12V_OUT: now also C20.+, X7.2
- net GND: now also C20.-, C21.-, C22.-, C23.-, D2.A, D3.A, IC10.2, IC10.4, IC5.3, IC5.5, IC5.6, IC7.1, R16.2, R20.1, X7.1; no longer D2.C, IC5.1, IC7.2
- net I_REF: now also IC7.2; no longer IC7.1
- net MISO: now also R21.2; no longer JP1.4
- net N$12: now also R20.2
- net N$18: now also Q4.C; no longer R16.2
- net N$27: now also JP1.4, R21.1; no longer Q4.C
Routing:
- net MISO: track 22.2 -> 0.00 mm
- net I_BATT: track 48.6 -> 68.5 mm
- net N$18: track 15.0 -> 34.1 mm
- net N$1: track 41.9 -> 58.2 mm
- net N$2: track 81.2 -> 92.5 mm
- net I_REF: track 74.0 -> 82.2 mm
- net +5V: track 134.7 -> 141.8 mm
- net N$27: track 6.35 -> 0.00 mm
- net 12V_OUT: track 69.7 -> 64.0 mm, vias 2 -> 1
- net +15V: track 211.6 -> 207.8 mm
- net N$12: track 28.1 -> 31.7 mm
- net N$28: track 3.43 -> 0.00 mm
- net N$24: track 0.00 -> 3.37 mm
- net N$3: track 12.1 -> 10.7 mm
- net N$4: track 6.35 -> 7.41 mm

Commit message: Add files via upload
Parts:
- moved R21 190.8 mm to (125.7, 20.3), turned to 90 degrees
- moved R16 180.9 mm to (118.1, 20.3), turned to 90 degrees
- moved IC1 11.4 mm to (123.8, 63.5)
- moved C10 1.27 mm to (86.4, 43.8)
- moved IC10 0.13 mm to (75.4, 42.5)
Routing:
- net N$27: track 0.00 -> 24.8 mm, vias 0 -> 2
- net I_BATT: track 68.5 -> 48.6 mm
- net N$1: track 58.2 -> 41.9 mm
- net N$2: track 92.5 -> 81.2 mm
- net I_REF: track 82.2 -> 74.0 mm
- net MISO: track 0.00 -> 5.40 mm
- net +15V: track 207.8 -> 211.7 mm
- net +5V: track 141.8 -> 144.1 mm
- net N$3: track 10.7 -> 9.36 mm
- net N$4: track 7.41 -> 7.93 mm

Commit message: Add files via upload
Parts:
- removed C17: (no value), rcl:E2,5-6
- removed JP2: (no value), pinhead:2X08
- removed X5: (no value), con-ptr500:AK500/2
- added C24: 1u, rcl:C0805
- added JP6, JP7, JP8: (no value), pinhead:1X08
- moved L1 237.0 mm to (16.5, 23.5), turned to 270 degrees
- moved D3 225.4 mm to (24.1, 40.6)
- moved R22 208.7 mm to (28.6, 34.3), turned to 90 degrees
- moved C21 204.1 mm to (10.8, 50.8), turned to 270 degrees
- moved C23 174.0 mm to (28.6, 8.89), turned to 270 degrees
- moved JP5 164.4 mm to (40.6, 14.6), flipped to the top, turned to 90 degrees
- moved C22 152.8 mm to (45.7, 27.9)
- moved IC5 136.4 mm to (26.0, 50.2), turned to 270 degrees
- moved C20 122.9 mm to (10.8, 64.1), turned to 270 degrees
- moved C8 14.6 mm to (46.4, 5.81)
- moved JP3 14.0 mm to (52.1, 14.7)
- moved C16 12.7 mm to (57.1, 28.0)
- moved X1 10.2 mm to (148.6, 80.6)
- moved X3 10.2 mm to (148.6, 46.4)
- moved X2 10.2 mm to (148.6, 63.5)
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Connections:
- net 5V_OUT: no longer C17.+, X5.2
- net 5V_OUT_B: now also C24.2
- net GND: now also C24.1, JP6.1, JP6.2, JP6.3, JP6.4, JP6.5, JP6.6, JP6.7, JP6.8, JP7.1, JP7.2, JP7.3, JP7.4, JP7.5, JP7.6, JP7.7, JP7.8, JP8.1, JP8.2, JP8.3, JP8.4, JP8.5, JP8.6, JP8.7, JP8.8; no longer C17.-, JP2.1, JP2.10, JP2.11, JP2.12, JP2.13, JP2.14, JP2.15, JP2.16, JP2.2, JP2.3, JP2.4, JP2.5, JP2.6, JP2.7, JP2.8, JP2.9, X5.1
Routing:
- net 5V_OUT_B: track 0.00 -> 75.2 mm
- net +15V: track 211.7 -> 261.2 mm
- net 5V_OUT: track 83.4 -> 54.0 mm
- net 12V_OUT: track 64.0 -> 92.2 mm
- net N$33: track 0.00 -> 19.3 mm
- net N$31: track 0.00 -> 18.1 mm
- net N$1: track 41.9 -> 34.1 mm
- net N$6: track 135.8 -> 130.8 mm
- net N$4: track 7.93 -> 11.1 mm
- net +5V: track 144.1 -> 141.3 mm
- net GND: track 4.69 -> 1.98 mm, vias 3 -> 207
- net N$3: track 9.36 -> 11.2 mm
- net N$22: track 8.26 -> 6.99 mm
- net N$21: track 8.26 -> 6.99 mm
- net N$20: track 8.26 -> 6.99 mm
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Other:
- board size 163 x 99 mm -> 154 x 99 mm

Commit message: Add files via upload
Parts:
- moved IC3 3.18 mm to (51.4, 48.9)
- moved C4 1.90 mm to (53.3, 54.6)
Routing:
- net +15V: track 261.2 -> 258.0 mm
- net 5V_OUT: track 54.0 -> 52.3 mm
Other:
- board text added: "5.2V"
Changed lines of the file:
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@@
 <text x="144.325" y="32.445" size="2.54" layer="51" font="vector" rot="R180">-</text>
 <text x="88" y="3" size="1.778" layer="51" font="vector">SUPPLY_BOARD_1.0</text>
-<text x="38.16" y="1.665" size="1.778" layer="51" font="vector">5.0V</text>
+<text x="38.16" y="1.665" size="1.778" layer="51" font="vector">5.2V</text>
 <text x="10.22" y="88.81" size="2.54" layer="51" font="vector" rot="R90">+</text>
 <text x="10.22" y="84.35" size="2.54" layer="51" font="vector" rot="R90">-</text>
@@
 <element name="C2" library="rcl" package="C0805" value="47n" x="122.555" y="41.275" rot="R270"/>
 <element name="C3" library="rcl" package="C0805" value="4n7" x="127" y="40.005" rot="R180"/>
-<element name="C4" library="rcl" package="C0805" value="1u" x="55.245" y="54.61" rot="R90"/>
+<element name="C4" library="rcl" package="C0805" value="1u" x="53.34" y="54.61" rot="R90"/>
 <element name="C5" library="rcl" package="E5-13" value="?" x="80.645" y="73.66"/>
 <element name="C6" library="rcl" package="C0805" value="1u" x="98.425" y="67.31" rot="R90"/>
@@
 </element>
 <element name="IC2" library="linear" package="DIL14" value="LM324N" x="98.425" y="57.15" rot="R180"/>
-<element name="IC3" library="linear" package="TO220V" value="AIMTEC 5.0V" x="48.26" y="48.895" rot="R270"/>
+<element name="IC3" library="linear" package="TO220V" value="AIMTEC 5.0V" x="51.435" y="48.895" rot="R270"/>
 <element name="IC4" library="linear" package="TO220V" value="AIMTEC 3.3V" x="66.04" y="48.895" rot="R270"/>
 <element name="IC6" library="mcp3208" package="DIL16" value="MCP3208" x="127" y="30.48" rot="R180"/>
@@
 <via x="38.1" y="81.28" extent="1-16" drill="0.3"/>
 <wire x1="38.1" y1="81.28" x2="38.1" y2="85.725" width="0.6604" layer="1"/>
-<wire x1="45.72" y1="51.435" x2="55.245" y2="51.435" width="1.5" layer="1"/>
-<wire x1="55.245" y1="51.435" x2="63.5" y2="51.435" width="1.5" layer="1"/>
-<wire x1="55.245" y1="53.66" x2="55.245" y2="51.435" width="1.5" layer="1"/>
+<wire x1="48.895" y1="51.435" x2="53.34" y2="51.435" width="1.5" layer="1"/>
+<wire x1="53.34" y1="51.435" x2="63.5" y2="51.435" width="1.5" layer="1"/>
+<wire x1="53.34" y1="53.66" x2="53.34" y2="51.435" width="1.5" layer="1"/>
 <contactref element="IC10" pad="1"/>
 <contactref element="IC5" pad="1"/>
@@
 <wire x1="47.305" y1="5.81" x2="52.07" y2="5.81" width="1.5" layer="1"/>
 <wire x1="52.07" y1="23.59" x2="52.07" y2="27.94" width="2" layer="1"/>
-<wire x1="52.07" y1="27.94" x2="52.07" y2="43.815" width="2" layer="1"/>
-<wire x1="52.07" y1="43.815" x2="49.53" y2="46.355" width="2" layer="1"/>
-<wire x1="49.53" y1="46.355" x2="45.72" y2="46.355" width="2" layer="1"/>
 <contactref element="C16" pad="+"/>
 <wire x1="55.88" y1="28.035" x2="52.165" y2="28.035" width="2" layer="1"/>
 <wire x1="52.165" y1="28.035" x2="52.07" y2="27.94" width="2" layer="1" curve="90"/>
+<wire x1="48.895" y1="46.355" x2="52.07" y2="46.355" width="2" layer="1"/>
+<wire x1="52.07" y1="46.355" x2="52.07" y2="27.94" width="2" layer="1"/>
 </signal>
 <signal name="3V3_OUT">
