File: schematics/tx_board_new/tx_board.sch (KiCad schematic (older format))
At the start: 45 parts, among them J1 Conn_02x14_Odd_Even, J301 Out, U301 ADF7021

Commit message: Add files via upload
Changed lines of the file:
@@
 Text GLabel 7100 8550 3    50   Input ~ 0
 ADF_CE
-Text GLabel 5700 8450 3    50   Input ~ 0
-FM_MOD
 Wire Wire Line
 	7800 8050 7800 7950
@@
 	1    7800 7950
 	-1   0    0    1
-$EndComp
-Wire Wire Line
-	8750 8300 8750 8400
-$Comp
-L power:GND #PWR010
-U 1 1 5F5D15A4
-P 8750 8400
-F 0 "#PWR010" H 8750 8150 50  0001 C CNN
-F 1 "GND" H 8755 8227 50  0000 C CNN
-F 2 "" H 8750 8400 50  0001 C CNN
-F 3 "" H 8750 8400 50  0001 C CNN
-	1    8750 8400
-	1    0    0    -1
 $EndComp
 Wire Wire Line
@@
 	1    7200 7950
 	-1   0    0    1
-$EndComp
-Wire Wire Line
-	5800 8450 5800 8550
-$Comp
-L power:GND #PWR06
-U 1 1 5F5E3E22
-P 5800 8550
-F 0 "#PWR06" H 5800 8300 50  0001 C CNN
-F 1 "GND" H 5805 8377 50  0000 C CNN
-F 2 "" H 5800 8550 50  0001 C CNN
-F 3 "" H 5800 8550 50  0001 C CNN
-	1    5800 8550
-	1    0    0    -1
-$EndComp
-Wire Wire Line
-	6550 8600 6550 8700
-$Comp
-L power:GND #PWR08
-U 1 1 5F5EA477
-P 6550 8700
-F 0 "#PWR08" H 6550 8450 50  0001 C CNN
-F 1 "GND" H 6555 8527 50  0000 C CNN
-F 2 "" H 6550 8700 50  0001 C CNN
-F 3 "" H 6550 8700 50  0001 C CNN
-	1    6550 8700
-	1    0    0    -1
 $EndComp
 Wire Wire Line
@@
 	8250 8550 8200 8550
 Wire Wire Line
-	5600 8450 5600 8550
-$Comp
-L power:GND #PWR02
-U 1 1 5F63542E
-P 5600 8550
-F 0 "#PWR02" H 5600 8300 50  0001 C CNN
-F 1 "GND" H 5605 8377 50  0000 C CNN
-F 2 "" H 5600 8550 50  0001 C CNN
-F 3 "" H 5600 8550 50  0001 C CNN
-	1    5600 8550
-	1    0    0    -1
-$EndComp
-Wire Wire Line
 	7000 8050 7000 7950
 $Comp
@@
 	7300 7950 7300 8050
 $Comp
-L power:+3.3V #PWR04
-U 1 1 5F65259F
-P 6400 8600
-F 0 "#PWR04" H 6400 8450 50  0001 C CNN
-F 1 "+3.3V" H 6415 8773 50  0000 C CNN
-F 2 "" H 6400 8600 50  0001 C CNN
-F 3 "" H 6400 8600 50  0001 C CNN
-	1    6400 8600
-	-1   0    0    1
-$EndComp
-Wire Wire Line
-	6400 8600 6400 8500
-$Comp
 L Connector_Generic:Conn_02x14_Odd_Even J1
